File: hardware/rev2/gadget_speed_radar_rev2.sch (KiCad schematic (older format))
At the start: 24 parts, among them P1 HB100, P2 MCU, U1 OPA2365, U2 MAX9031

Commit message: ordered pcbs
Parts:
- added C10: 100nF, Capacitors_SMD:C_0805, symbol C
- added R11: 47K, Resistors_SMD:R_0805, symbol R
- added R9: 1K, Resistors_SMD:R_0805, symbol R
- C1, C2, C3, C4, C5, C6, C7, C8, C9: footprint (none) -> Capacitors_SMD:C_0805
- FB1, R1, R10, R2, R3, R4, R5, R6, R7, R8: footprint (none) -> Resistors_SMD:R_0805
- P1, P2: footprint (none) -> Connectors_Molex:Molex_KK-6410-03_03x2.54mm_Straight
- RV1: footprint (none) -> Potentiometers:Potentiometer_Trimmer-Suntan-TSR-3386P
- U1: footprint (none) -> Housings_SOIC:SOIC-8_3.9x4.9mm_Pitch1.27mm
- U2: footprint (none) -> TO_SOT_Packages_SMD:SOT-23-5
Connections:
- net GND: now also C10.2
- net at C2.1, FB1.1, R2.1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: now also C10.1
- net at R10.1, RV1.2, RV1.3: now also R9.1; no longer U2.1 (IN+)
- net at P2.2 (P2), U2.4 (OUT): now also R11.1
- new net: R11.2, R9.2, U2.1 (IN+)
Other:
- note added: "100mV hysteresis"
- moved on the sheet: P2, R10
